File: модуль стойки/module/module.kicad_pcb (KiCad board)
At the start: 2 copper layers, 33 x 16 mm, 7 parts

Commit message: модуль на стадии редактировании
Parts:
- removed XS1, XS2, XS3, XS4, XS5: отверстие_под_пайку, MOTOR_ICO:Отверстие_под_пайку_D1.2
- added C1: Конденсатор_керамический, MOTOR_RLC:Конденсатор_SMD_1812, B.Cu at (151.0, 78.5)
- added C2: Конденсатор_керамический, MOTOR_RLC:Конденсатор_SMD_1812, B.Cu at (152.5, 89.5)
- added C3: Конденсатор_керамический, MOTOR_RLC:Конденсатор_SMD_1812, B.Cu at (139.0, 88.5)
- added FU1: Предохранитель, N_RLC:Предохранитель_R700, F.Cu at (142.5, 94.5)
- moved VT2 9.05 mm to (139.0, 83.0)
- moved VT1 6.91 mm to (152.5, 83.5)
Routing:
- net Net-(C2-Pad2): track 27.3 -> 0.00 mm
- net Net-(C3-Pad1): track 25.8 -> 0.00 mm
- net Net-(C2-Pad1): track 18.3 -> 0.00 mm
- net Net-(C1-Pad2): track 15.9 -> 0.00 mm
- net Net-(C1-Pad1): track 7.74 -> 0.00 mm
Other:
- board size 33 x 16 mm -> 35 x 16 mm
- net class Default: clearance 0.2 -> 0.4; trace_width 0.5 -> 0.4
- net class СИЛА added: clearance 0.4, trace_width 2.4, via_dia 0.8, via_drill 0.4
- rule trace_clearance: 0.2 -> 0.4

Commit message: нет индикации
Parts:
- C1, C2, C3: footprint MOTOR_RLC:Конденсатор_SMD_1812 -> N_RLC:Конденсатор_SMD_2220
- VT1: footprint MOTOR_IMPORT_OTK:Транзистор_P_IRF9Z24NPBF -> N_DD:SO-8
- VT2: footprint MOTOR_IMPORT_OTK:Транзистор_N_STP10NK60Z -> N_DD:SO-8
- moved FU1 30.8 mm to (121.5, 72.0)
- moved VT1 15.2 mm to (158.5, 69.5)
- moved VT2 13.2 mm to (141.5, 70.0)

Commit message: модуль стойки - готов
без индикации
Parts:
- removed C1, C2: Конденсатор_керамический, N_RLC:Конденсатор_SMD_2220
- added R1: Резистор_0,125Вт, N_RLC:Резистор_SMD_0805_0,125Вт, F.Cu at (202.5, 86.0)
- added R2: Резистор_0,125Вт, N_RLC:Резистор_SMD_0805_0,125Вт, F.Cu at (202.5, 83.0)
- added R3: Резистор_0,125Вт, N_RLC:Резистор_SMD_0805_0,125Вт, F.Cu at (202.5, 80.0)
- added R4: Резистор_0,125Вт, N_RLC:Резистор_SMD_0805_0,125Вт, F.Cu at (212.0, 94.0)
- added VT3: Транзистор_полевой_P-канал, MOTOR_IMPORT_OTK:Транзистор_P_IRF9Z24NPBF, F.Cu at (214.5, 76.5)
- added VT4: Транзистор_полевой_N-канал, MOTOR_IMPORT_OTK:Транзистор_N_STP10NK60Z, F.Cu at (219.0, 82.2)
- added XP1: Вилка_PLS8, N_X:Вилка_PLS8_вертикальная, F.Cu at (199.5, 76.0)
- added XP2: Вилка_PLS6, N_X:Вилка_PLS6_вертикальная, F.Cu at (234.5, 73.5)
- added rM3: Отверстие_М3, N_X:Отверстие_М3, F.Cu at (231.5, 95.0)
- C3: footprint N_RLC:Конденсатор_SMD_2220 -> MOTOR_RLC:Конденсатор_SMD_1812; moved to F.Cu
- FU1: footprint N_RLC:Предохранитель_R700 -> N_RLC:Предохранитель_MF-R_d10.4
- VT1: value Транзистор_полевой_P-канал -> Транзистор_полевой_P-канал(so-8)
- VT2: value Транзистор_полевой_N-канал -> Транзистор_полевой_N-канал(so-8)
- moved C3 85.2 mm to (224.0, 94.0), turned to 180 degrees
- moved FU1 83.5 mm to (205.0, 72.5)
- moved VT2 73.1 mm to (213.0, 85.0)
- moved VT1 70.6 mm to (227.0, 86.5)
Connections:
- C3 pad 2: Net-(C1-Pad2) -> Net-(C3-Pad2)
- FU1 pad 1: Net-(C2-Pad2) -> Net-(FU1-Pad1)
- FU1 pad 2: Net-(FU1-Pad2) -> Net-(C3-Pad1)
- VT1 pad 1: Net-(C2-Pad1) -> Net-(C3-Pad1)
- VT1 pad 3: Net-(C2-Pad2) -> Net-(C3-Pad1)
- VT1 pad 4: (no net) -> Net-(R2-Pad2)
- VT1 pad 5: (no net) -> Net-(VT1-Pad5)
- VT1 pad 6: (no net) -> Net-(VT1-Pad5)
- VT1 pad 7: (no net) -> Net-(VT1-Pad5)
- VT1 pad 8: (no net) -> Net-(VT1-Pad5)
- VT2 pad 1: Net-(C1-Pad1) -> Net-(C3-Pad2)
- VT2 pad 2: Net-(C2-Pad2) -> Net-(C3-Pad2)
- VT2 pad 3: Net-(C1-Pad2) -> Net-(C3-Pad2)
- VT2 pad 4: (no net) -> Net-(R1-Pad2)
- VT2 pad 5: (no net) -> Net-(VT1-Pad5)
- VT2 pad 6: (no net) -> Net-(VT1-Pad5)
- VT2 pad 7: (no net) -> Net-(VT1-Pad5)
- VT2 pad 8: (no net) -> Net-(VT1-Pad5)
Routing:
- net Net-(R2-Pad2): track 0.00 -> 47.8 mm, vias 0 -> 2
- net Net-(R1-Pad2): track 0.00 -> 40.7 mm, vias 0 -> 2
- net Net-(C3-Pad1): track 0.00 -> 12.1 mm, vias 0 -> 2
- net Net-(C3-Pad2): track 0.00 -> 10.6 mm
- net Net-(R2-Pad1): track 0.00 -> 3.26 mm
- net Net-(R1-Pad1): track 0.00 -> 3.07 mm
- net Net-(VT1-Pad5): track 0.00 -> 2.54 mm
- added copper zone on B.Cu, net Net-(C3-Pad1)
- added copper zone on F.Cu, net Net-(C3-Pad1)
- added copper zone on F.Cu, net Net-(C3-Pad2)
- added copper zone on B.Cu, net Net-(FU1-Pad1)
- added copper zone on F.Cu, net Net-(VT1-Pad5)
Other:
- board size 35 x 16 mm -> 40 x 30 mm
- net class Default: trace_width 0.4 -> 1
- net class СИЛА: trace_width 2.4 -> 1
- net class управление added: clearance 0.4, trace_width 0.4, via_dia 0.8, via_drill 0.4
- rule trace_min: 0.2 -> 0.4

Commit message: Платы
Parts:
- added HL1: Светодиод, N_VD_HL:Светодиод_SMD_0603, F.Cu at (205.5, 97.5)
- added R5: Резистор_0,125Вт, N_RLC:Резистор_SMD_0805_0,125Вт, F.Cu at (203.5, 92.5)
- moved rM3 0.50 mm to (232.0, 95.0)
Routing:
- net Net-(C3-Pad1): track 12.1 -> 21.4 mm, vias 2 -> 3
- net Net-(HL1-Pad1): track 0.00 -> 5.00 mm
Other:
- board text added: "hb.0"
Changed lines of the file:
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@@
   (general
     (thickness 1.6)
-    (drawings 4)
-    (tracks 48)
+    (drawings 5)
+    (tracks 54)
     (zones 0)
-    (modules 13)
-    (nets 9)
+    (modules 15)
+    (nets 10)
   )
   (page A4)
@@
     (35 F.Paste user)
     (36 B.SilkS user)
-    (37 F.SilkS user)
+    (37 F.SilkS user hide)
     (38 B.Mask user)
     (39 F.Mask user)
@@
     (visible_elements 7FFFFFFF)
     (pcbplotparams
-      (layerselection 0x010fc_ffffffff)
+      (layerselection 0x010c0_ffffffff)
       (usegerberextensions false)
       (usegerberattributes false)
@@
       (outputformat 1)
       (mirror false)
-      (drillshape 1)
+      (drillshape 0)
       (scaleselection 1)
-      (outputdirectory ""))
+      (outputdirectory "gerber/"))
   )
   (net 0 "")
@@
   (net 7 "Net-(R2-Pad2)")
   (net 8 "Net-(VT1-Pad5)")
+  (net 9 "Net-(HL1-Pad1)")
   (net_class Default "Это класс цепей по умолчанию."
     (clearance 0.4)
@@
     (add_net "Net-(C3-Pad2)")
     (add_net "Net-(FU1-Pad1)")
+    (add_net "Net-(HL1-Pad1)")
     (add_net "Net-(VT1-Pad5)")
   )
@@
   )
   (module N_X:Отверстие_М3 (layer F.Cu)
-    (at 231.5 95)
+    (at 232 95)
     (fp_text reference rM3 (at -4.5 3.5) (layer F.SilkS) hide
       (effects (font (size 1.5 1.5) (thickness 0.15)))
@@
       (net 5 "Net-(C3-Pad2)"))
   )
+  (module N_VD_HL:Светодиод_SMD_0603 (layer F.Cu)
+    (at 205.5 97.5 180)
+    (fp_text reference HL1 (at 0.5 2 180) (layer F.SilkS)
+      (effects (font (size 1 1) (thickness 0.2)))
+    )
+    (fp_text value Светодиод (at 0.1524 2.5146 180) (layer F.Fab)
+      (effects (font (size 1 1) (thickness 0.15)))
+    )
+    (fp_line (start -0.9 -0.9) (end -0.9 0.9) (layer F.SilkS) (width 0.3))
+    (fp_line (start -0.9 -0.9) (end -0.4 -0.9) (layer F.SilkS) (width 0.3))
+    (fp_line (start -0.9 0.9) (end -0.4 0.9) (layer F.SilkS) (width 0.3))
+    (fp_line (start 2.4 0.9) (end 1.9 0.9) (layer F.SilkS) (width 0.3))
+    (fp_line (start 2.4 0.9) (end 2.4 -0.6) (layer F.SilkS) (width 0.3))
+    (fp_line (start 1.9 -0.9) (end 2.1 -0.9) (layer F.SilkS) (width 0.3))
+    (fp_line (start 2.1 -0.9) (end 2.4 -0.6) (layer F.SilkS) (width 0.3))
+    (pad 1 smd rect (at 0 0 180) (size 1 1) (layers F.Cu F.Paste F.Mask)
+      (net 9 "Net-(HL1-Pad1)") (clearance 0.2))
+    (pad 2 smd rect (at 1.5 0 180) (size 1 1) (layers F.Cu F.Paste F.Mask)
+      (net 5 "Net-(C3-Pad2)") (clearance 0.2))
+    (model ${N_3D}/LED_0603.step
+      (offset (xyz 0.75 0 0))
+      (scale (xyz 1 1 1))
+      (rotate (xyz 0 0 0))
+    )
+  )
+  (module N_RLC:Резистор_SMD_0805_0,125Вт (layer F.Cu)
+    (at 203.5 92.5)
+    (fp_text reference R5 (at 1 -2) (layer F.SilkS)
+      (effects (font (size 1 1) (thickness 0.2)))
+    )
+    (fp_text value Резистор_0,125Вт (at 1.29 2.09) (layer F.Fab) hide
+      (effects (font (size 2 1.6) (thickness 0.3)))
+    )
+    (fp_line (start -0.6 1.15) (end -0.1 1.15) (layer F.SilkS) (width 0.3))
+    (fp_line (start 2.5 1.15) (end 2 1.15) (layer F.SilkS) (width 0.3))
+    (fp_line (start -0.9 -1.15) (end 0.1 -1.15) (layer F.SilkS) (width 0.3))
+    (fp_line (start 2.9 -1.15) (end 1.9 -1.15) (layer F.SilkS) (width 0.3))
+    (fp_line (start 2.9 1.15) (end 1.9 1.15) (layer F.SilkS) (width 0.3))
+    (fp_line (start -0.9 1.15) (end 0.1 1.15) (layer F.SilkS) (width 0.3))
+    (fp_line (start 2.9 -1.15) (end 2.9 1.15) (layer F.SilkS) (width 0.3))
+    (fp_line (start -0.9 1.15) (end -0.9 -1.15) (layer F.SilkS) (width 0.3))
+    (fp_line (start 0.85 -0.45) (end 1.15 -0.2) (layer F.SilkS) (width 0.3))
+    (fp_line (start 0.85 0.2) (end 1.15 0.45) (layer F.SilkS) (width 0.3))
+    (pad 2 smd rect (at 2 0) (size 1 1.5) (layers F.Cu F.Paste F.Mask)
+      (net 9 "Net-(HL1-Pad1)") (clearance 0.2))
+    (pad 1 smd rect (at 0 0) (size 1 1.5) (layers F.Cu F.Paste F.Mask)
+      (net 1 "Net-(C3-Pad1)") (clearance 0.2))
+    (model ${N_3D}/Res_0805.stp
+      (offset (xyz 0.05 0.61 0))
+      (scale (xyz 1 1 1))
+      (rotate (xyz 0 0 90))
+    )
+  )
+  (gr_text hb.0 (at 227.5 74) (layer F.Cu)
+    (effects (font (size 1 1) (thickness 0.25)))
+  )
   (gr_line (start 237 100) (end 237 70) (angle 90) (layer Edge.Cuts) (width 0.15))
   (gr_line (start 197 100) (end 237 100) (angle 90) (layer Edge.Cuts) (width 0.15))
@@
   (via (at 232.5 88.5) (size 0.8) (drill 0.4) (layers F.Cu B.Cu) (net 1))
   (via (at 231 88.5) (size 0.8) (drill 0.4) (layers F.Cu B.Cu) (net 1))
+  (segment (start 203.5 90.75) (end 204.25 90) (width 1) (layer F.Cu) (net 1))
+  (segment (start 203.5 92.5) (end 203.5 90.75) (width 1) (layer F.Cu) (net 1))
+  (via (at 210.5 90.5) (size 0.8) (drill 0.4) (layers F.Cu B.Cu) (net 1))
+  (segment (start 204.25 90) (end 210 90) (width 1) (layer F.Cu) (net 1))
+  (segment (start 210 90) (end 210.5 90.5) (width 1) (layer F.Cu) (net 1))
   (segment (start 199.5 86.16) (end 202.34 86.16) (width 0.4) (layer F.Cu) (net 2) (status C00000))
   (segment (start 202.34 86.16) (end 202.5 86) (width 0.4) (layer F.Cu) (net 2) (status C00000))
@@
   (segment (start 228 92) (end 228.905 91.095) (width 0.4) (layer F.Cu) (net 7))
   (segment (start 234.5 86.2) (end 234.5 83.66) (width 1) (layer F.Cu) (net 8))
+  (segment (start 205.5 97.5) (end 205.5 92.5) (width 1) (layer F.Cu) (net 9))
   (zone (net 8) (net_name "Net-(VT1-Pad5)") (layer F.Cu) (hatch edge 0.508)
     (connect_pads (clearance 0.5))
