File: модуль стойки/module/module.sch (KiCad schematic (older format))
At the start: 7 parts

Commit message: модуль на стадии редактировании
Parts:
- removed XS1, XS2, XS3, XS4, XS5: отверстие_под_пайку, MOTOR_ICO:Отверстие_под_пайку_D1.2, symbol MOTOR:отверстие_под_пайку
- added C1, C2, C3: Конденсатор_керамический, MOTOR_RLC:Конденсатор_SMD_1812, symbol elements:Конденсатор_керамический
- added FU1: Предохранитель, N_RLC:Предохранитель_R700, symbol elements:Предохранитель
- added XP1: Вилка_PLS8, symbol elements:Вилка_PLS8
- added XP2: Вилка_PLS6, symbol elements:Вилка_PLS6
- VT2: symbol MOTOR:Транзистор_полевой_N-канал -> elements:Транзистор_полевой_N-канал
Connections:
- wire segments 13 -> 59
- no-connect marks 0 -> 1
Changed lines of the file:
@@
 $EndDescr
 $Comp
-L MOTOR:Транзистор_полевой_N-канал VT2
+L elements:Транзистор_полевой_N-канал VT2
 U 1 1 5C236B1C
 P 4700 3850
@@
 	1    0    0    -1
 $EndComp
-$Comp
-L MOTOR:отверстие_под_пайку XS1
-U 1 1 5C236D99
-P 2900 2500
-F 0 "XS1" H 2940 2578 60  0000 L CNN
-F 1 "отверстие_под_пайку" H 2940 2472 60  0000 L CNN
-F 2 "MOTOR_ICO:Отверстие_под_пайку_D1.2" H 2900 2500 60  0001 C CNN
-F 3 "" H 2900 2500 60  0001 C CNN
-	1    2900 2500
-	1    0    0    -1
-$EndComp
-$Comp
-L MOTOR:отверстие_под_пайку XS2
-U 1 1 5C236DF4
-P 2950 3200
-F 0 "XS2" H 2990 3278 60  0000 L CNN
-F 1 "отверстие_под_пайку" H 2990 3172 60  0000 L CNN
-F 2 "MOTOR_ICO:Отверстие_под_пайку_D1.2" H 2950 3200 60  0001 C CNN
-F 3 "" H 2950 3200 60  0001 C CNN
-	1    2950 3200
-	1    0    0    -1
-$EndComp
-$Comp
-L MOTOR:отверстие_под_пайку XS3
-U 1 1 5C236E57
-P 2950 3850
-F 0 "XS3" H 2990 3928 60  0000 L CNN
-F 1 "отверстие_под_пайку" H 2990 3822 60  0000 L CNN
-F 2 "MOTOR_ICO:Отверстие_под_пайку_D1.2" H 2950 3850 60  0001 C CNN
-F 3 "" H 2950 3850 60  0001 C CNN
-	1    2950 3850
-	1    0    0    -1
-$EndComp
-$Comp
-L MOTOR:отверстие_под_пайку XS4
-U 1 1 5C236EBA
-P 2950 4600
-F 0 "XS4" H 2990 4678 60  0000 L CNN
-F 1 "отверстие_под_пайку" H 2990 4572 60  0000 L CNN
-F 2 "MOTOR_ICO:Отверстие_под_пайку_D1.2" H 2950 4600 60  0001 C CNN
-F 3 "" H 2950 4600 60  0001 C CNN
-	1    2950 4600
-	1    0    0    -1
-$EndComp
-Wire Wire Line
-	2950 3850 4450 3850
 $Comp
 L elements:Транзистор_полевой_P-канал VT1
@@
 	3750 3200 3750 3050
 Wire Wire Line
-	3750 3050 4450 3050
+	3750 3050 4050 3050
 Wire Wire Line
 	2900 2500 5250 2500
@@
 	5250 2500 5250 2750
 Wire Wire Line
-	2950 4600 5250 4600
-Wire Wire Line
 	5250 4600 5250 3850
-$Comp
-L MOTOR:отверстие_под_пайку XS5
-U 1 1 5C23A0C2
-P 5850 3350
-F 0 "XS5" H 5890 3428 60  0000 L CNN
-F 1 "отверстие_под_пайку" H 5890 3322 60  0000 L CNN
-F 2 "MOTOR_ICO:Отверстие_под_пайку_D1.2" H 5850 3350 60  0001 C CNN
-F 3 "" H 5850 3350 60  0001 C CNN
-	1    5850 3350
-	1    0    0    -1
-$EndComp
-Wire Wire Line
-	5850 3350 5350 3350
+Wire Wire Line
+	7400 3700 7300 3700
 Connection ~ 5350 3350
 Wire Wire Line
 	5350 3350 5350 3050
+$Comp
+L elements:Конденсатор_керамический C3
+U 1 1 5C25C9F8
+P 6500 3500
+F 0 "C3" V 6472 3588 60  0000 L CNN
+F 1 "Конденсатор_керамический" V 6578 3588 60  0000 L CNN
+F 2 "MOTOR_RLC:Конденсатор_SMD_1812" H 6500 3500 60  0001 C CNN
+F 3 "" H 6500 3500 60  0001 C CNN
+	1    6500 3500
+	0    1    1    0
+$EndComp
+Wire Wire Line
+	5250 4600 6500 4600
+Wire Wire Line
+	6500 4600 6500 3600
+Connection ~ 5250 4600
+Wire Wire Line
+	6500 3450 6500 2500
+Wire Wire Line
+	6500 2500 5250 2500
+Connection ~ 5250 2500
+$Comp
+L elements:Конденсатор_керамический C1
+U 1 1 5C25CC91
+P 3950 4200
+F 0 "C1" V 3922 4288 60  0000 L CNN
+F 1 "Конденсатор_керамический" V 4028 4288 60  0000 L CNN
+F 2 "MOTOR_RLC:Конденсатор_SMD_1812" H 3950 4200 60  0001 C CNN
+F 3 "" H 3950 4200 60  0001 C CNN
+	1    3950 4200
+	0    1    1    0
+$EndComp
+Wire Wire Line
+	3950 4150 3950 3850
+Connection ~ 3950 3850
+Wire Wire Line
+	3950 3850 4450 3850
+Wire Wire Line
+	3950 4300 3950 4600
+Connection ~ 3950 4600
+Wire Wire Line
+	3950 4600 5250 4600
+$Comp
+L elements:Конденсатор_керамический C2
+U 1 1 5C25D02F
+P 4050 3150
+F 0 "C2" V 4022 3238 60  0000 L CNN
+F 1 "Конденсатор_керамический" V 4128 3238 60  0000 L CNN
+F 2 "MOTOR_RLC:Конденсатор_SMD_1812" H 4050 3150 60  0001 C CNN
+F 3 "" H 4050 3150 60  0001 C CNN
+	1    4050 3150
+	0    1    1    0
+$EndComp
+Wire Wire Line
+	4050 3100 4050 3050
+Connection ~ 4050 3050
+Wire Wire Line
+	4050 3050 4450 3050
+Wire Wire Line
+	4050 3250 4050 3350
+Wire Wire Line
+	4050 3350 5350 3350
+Wire Wire Line
+	7300 3700 7300 3950
+Wire Wire Line
+	7300 3950 7400 3950
+NoConn ~ 4600 2900
+Wire Wire Line
+	2550 2850 2900 2850
+Wire Wire Line
+	2900 2850 2900 2500
+Wire Wire Line
+	2900 2950 2900 2850
+Connection ~ 2900 2850
+Wire Wire Line
+	2950 3050 2950 3200
+Wire Wire Line
+	2750 3150 2750 3850
+Wire Wire Line
+	2750 3850 3950 3850
+Wire Wire Line
+	2700 3250 2700 4600
+Wire Wire Line
+	2550 3350 2550 3450
+Wire Wire Line
+	2550 4600 2700 4600
+Connection ~ 2700 4600
+Wire Wire Line
+	2700 4600 3950 4600
+$Comp
+L elements:Вилка_PLS8 XP1
+U 1 1 5C262672
+P 1950 2650
+F 0 "XP1" H 2206 2731 60  0000 C CNN
+F 1 "Вилка_PLS8" H 2200 1700 60  0001 C CNN
+F 2 "" H 1950 2650 60  0001 C CNN
+F 3 "" H 1950 2650 60  0001 C CNN
+	1    1950 2650
+	1    0    0    -1
+$EndComp
+Wire Wire Line
+	2450 2750 2550 2750
+Wire Wire Line
+	2550 2750 2550 2850
+Wire Wire Line
+	2450 2850 2550 2850
+Connection ~ 2550 2850
+Wire Wire Line
+	2450 2950 2900 2950
+Wire Wire Line
+	2450 3050 2950 3050
+Wire Wire Line
+	2450 3150 2750 3150
+Wire Wire Line
+	2450 3250 2700 3250
+Wire Wire Line
+	2450 3350 2550 3350
+Wire Wire Line
+	2450 3450 2550 3450
+Connection ~ 2550 3450
+Wire Wire Line
+	2550 3450 2550 4600
+$Comp
+L elements:Вилка_PLS6 XP2
+U 1 1 5C267DB0
+P 7950 3500
+F 0 "XP2" H 7922 3163 60  0000 R CNN
+F 1 "Вилка_PLS6" H 8250 2725 60  0001 C CNN
+F 2 "" H 7950 3500 60  0001 C CNN
+F 3 "" H 7950 3500 60  0001 C CNN
+	1    7950 3500
+	-1   0    0    -1
+$EndComp
+Wire Wire Line
+	7400 3700 7400 3600
+Wire Wire Line
+	7400 3600 7450 3600
+Wire Wire Line
+	7400 3700 7450 3700
+Connection ~ 7400 3700
+Wire Wire Line
+	7400 3950 7400 3900
+Wire Wire Line
+	7400 3800 7450 3800
+Wire Wire Line
+	7450 3900 7400 3900
+Connection ~ 7400 3900
+Wire Wire Line
+	7400 3900 7400 3800
+Wire Wire Line
+	7450 4000 7400 4000
+Wire Wire Line
+	7400 4000 7400 3950
+Connection ~ 7400 3950
+Wire Wire Line
+	7450 4100 7400 4100
+Wire Wire Line
+	7400 4100 7400 4000
+Connection ~ 7400 4000
+$Comp
+L elements:Предохранитель FU1
+U 1 1 5C26F005
+P 6000 3350
+F 0 "FU1" H 6000 3612 60  0000 C CNN
+F 1 "Предохранитель" H 6000 3506 60  0000 C CNN
+F 2 "N_RLC:Предохранитель_R700" H 6000 3350 60  0001 C CNN
+F 3 "" H 6000 3350 60  0001 C CNN
+	1    6000 3350
+	1    0    0    -1
+$EndComp
+Wire Wire Line
+	5350 3350 5600 3350
+Wire Wire Line
+	6400 3350 7300 3350
+Wire Wire Line
+	7300 3350 7300 3700
+Connection ~ 7300 3700
 $EndSCHEMATC

Commit message: модуль стойки - готов
без индикации
Parts:
- removed C1, C2: Конденсатор_керамический, MOTOR_RLC:Конденсатор_SMD_1812, symbol elements:Конденсатор_керамический
- removed VT1: Транзистор_полевой_P-канал, MOTOR_IMPORT_OTK:Транзистор_P_IRF9Z24NPBF, symbol elements:Транзистор_полевой_P-канал
- removed VT2: Транзистор_полевой_N-канал, MOTOR_IMPORT_OTK:Транзистор_N_STP10NK60Z, symbol elements:Транзистор_полевой_N-канал
- added R1, R2, R3, R4: Резистор_0,125Вт, N_RLC:Резистор_SMD_0805_0,125Вт, symbol elements:Резистор_0,125Вт
- added VT1: Транзистор_полевой_P-канал(so-8), N_DD:SO-8, symbol elements:Транзистор_полевой_P-канал(so-8)
- added VT2: Транзистор_полевой_N-канал(so-8), N_DD:SO-8, symbol elements:Транзистор_полевой_N-канал(so-8)
- added VT3: Транзистор_полевой_P-канал, MOTOR_IMPORT_OTK:Транзистор_P_IRF9Z24NPBF, symbol elements:Транзистор_полевой_P-канал
- added VT4: Транзистор_полевой_N-канал, MOTOR_IMPORT_OTK:Транзистор_N_STP10NK60Z, symbol elements:Транзистор_полевой_N-канал
- FU1: footprint N_RLC:Предохранитель_R700 -> N_RLC:Предохранитель_MF-R_d10.4
- XP1: footprint (none) -> N_X:Вилка_PLS8_вертикальная
- XP2: footprint (none) -> N_X:Вилка_PLS6_вертикальная
Connections:
- wire segments 59 -> 86
- no-connect marks 1 -> 0

Commit message: Платы
Parts:
- added HL1: Светодиод, N_VD_HL:Светодиод_SMD_0603, symbol elements:Светодиод
- added R5: Резистор_0,125Вт, N_RLC:Резистор_SMD_0805_0,125Вт, symbol elements:Резистор_0,125Вт
Connections:
- wire segments 86 -> 91
Changed lines of the file:
@@
 Wire Wire Line
 	6300 4600 6500 4600
+$Comp
+L elements:Светодиод HL1
+U 1 1 5C3F6AD0
+P 7350 2100
+F 0 "HL1" H 7500 2412 60  0000 C CNN
+F 1 "Светодиод" H 7500 2306 60  0000 C CNN
+F 2 "N_VD_HL:Светодиод_SMD_0603" H 7650 1600 60  0001 C CNN
+F 3 "" H 7650 1600 60  0001 C CNN
+	1    7350 2100
+	1    0    0    -1
+$EndComp
+$Comp
+L elements:Резистор_0,125Вт R5
+U 1 1 5C3F6DAB
+P 6850 2100
+F 0 "R5" H 6850 2362 60  0000 C CNN
+F 1 "Резистор_0,125Вт" H 6850 2256 60  0000 C CNN
+F 2 "N_RLC:Резистор_SMD_0805_0,125Вт" H 6850 2100 60  0001 C CNN
+F 3 "" H 6850 2100 60  0001 C CNN
+	1    6850 2100
+	1    0    0    -1
+$EndComp
+Wire Wire Line
+	6300 2100 6450 2100
+Connection ~ 6300 2100
+Wire Wire Line
+	7250 2100 7350 2100
+Wire Wire Line
+	7650 2100 8400 2100
+Wire Wire Line
+	8400 2100 8400 4600
+Wire Wire Line
+	8400 4600 6500 4600
+Connection ~ 6500 4600
 $EndSCHEMATC
